Commit message: before project protection

File: src/robot_description/urdf/park_robot.urdf (robot description, URDF)
Before this commit: robot park_robot, 3 links, 2 joints
Links:
- removed link base_footprint
- removed link laser_frame
- link base_link: geometry visual box size=0.5 0.5 0.5
Joints:
- removed joint base_footprint_to_base_link
- removed joint base_link_to_laser
